File: aix_amp/aix_amp.kicad_sch (KiCad schematic)
At the start: 0 parts

Commit message: add interface
Other:
- added sheet filter (filter.kicad_sch)
- added sheet interface (interface.kicad_sch)
Changed lines of the file:
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@@
 	(paper "A4")
 	(sheet
-		(at 67.31 20.32)
+		(at 21.59 52.07)
+		(size 36.83 33.02)
+		(exclude_from_sim no)
+		(in_bom yes)
+		(on_board yes)
+		(dnp no)
+		(fields_autoplaced yes)
+		(stroke
+			(width 0.1524)
+			(type solid)
+		)
+		(fill
+			(color 0 0 0 0.0000)
+		)
+		(property "Sheetname" "interface"
+			(at 21.59 51.3584 0)
+			(effects
+				(font
+					(size 1.27 1.27)
+				)
+				(justify left bottom)
+			)
+		)
+		(property "Sheetfile" "interface.kicad_sch"
+			(at 21.59 85.6746 0)
+			(effects
+				(font
+					(size 1.27 1.27)
+				)
+				(justify left top)
+			)
+		)
+		(instances
+			(project "aix_amp"
+				(path "/92363970-7a70-4a9d-91f1-fb8480a3037e"
+					(page "5")
+				)
+			)
+		)
+	)
+	(sheet
+		(at 67.31 55.88)
 		(size 69.85 20.32)
 		(exclude_from_sim no)
@@
 		)
 		(property "Sheetname" "amp"
-			(at 67.31 19.6084 0)
+			(at 67.31 55.1684 0)
 			(effects
 				(font
@@
 		)
 		(property "Sheetfile" "amp.kicad_sch"
-			(at 67.31 41.2246 0)
+			(at 67.31 76.7846 0)
 			(effects
 				(font
@@
 				)
 			)
+		)
+	)
+	(sheet
+		(at 67.31 20.32)
+		(size 69.85 22.86)
+		(exclude_from_sim no)
+		(in_bom yes)
+		(on_board yes)
+		(dnp no)
+		(fields_autoplaced yes)
+		(stroke
+			(width 0.1524)
+			(type solid)
+		)
+		(fill
+			(color 0 0 0 0.0000)
+		)
+		(property "Sheetname" "filter"
+			(at 67.31 19.6084 0)
+			(effects
+				(font
+					(size 1.27 1.27)
+				)
+				(justify left bottom)
+			)
+		)
+		(property "Sheetfile" "filter.kicad_sch"
+			(at 67.31 43.7646 0)
+			(effects
+				(font
+					(size 1.27 1.27)
+				)
+				(justify left top)
+			)
+		)
+		(instances
+			(project "aix_amp"
+				(path "/92363970-7a70-4a9d-91f1-fb8480a3037e"
+					(page "4")
+				)
+			)
