File: aix_amp/amp.kicad_sch (KiCad schematic)
At the start: 0 parts

Commit message: 앰프 기본 완성
Parts:
- added C8: 10uf, symbol Device:C
- added R16, R19, R21, R22: 12k, symbol Device:R_US
- added R17, R18, R20, R23: 2k, symbol Device:R_US
- added U1: Opamp_Quad, symbol Device:Opamp_Quad
Connections:
- new net: R16.2, R17.1, U1.9 (-)
- new net: R17.2, U1.5 (+), U1.8
- new net: R20.1, R21.2, U1.2 (-)
- new net: R20.2, U1.1
- new net: R23.2, U1.14, U1.3 (+)
- new net: R22.2, R23.1, U1.13 (-)
- new net: R18.1, R19.2, U1.6 (-)
- new net: R18.2, U1.7
- new net: C8.2, U1.4 (V+)
- new net +5V: C8.1
- new net GND: R16.1, R19.1, R21.1, R22.1, U1.11 (V-)
