File: aix_amp/filter.kicad_sch (KiCad schematic)
At the start: 0 parts

Commit message: 앰프 기본 완성
Parts:
- added C2, C3, C5, C6, C7: C, symbol Device:C
- added R10, R11, R3, R4: R_US, symbol Device:R_US
- added SW1: SW_DPDT_x2, Button_Switch_THT:SW_CK_JS202011AQN_DPDT_Angled, symbol Switch:SW_DPDT_x2
- added U5: Opamp_Dual, symbol Device:Opamp_Dual
Connections:
- new net: C2.2, C3.1, R4.1, U5.3 (+)
- new net: C3.2, R4.2, SW1.1 (A), U5.1
- new net: R10.1, SW1.6 (C)
- new net: C5.1, R10.2
- new net: C5.2, C6.1, R11.1, U5.5 (+)
- new net: C6.2, R11.2, SW1.4 (A), U5.7
- new net: C7.2, U5.8 (V+)
- new net: C2.1, R3.2
- new net: R3.1, SW1.3 (C)
- new net +5V: C7.1
- new net GND: U5.2 (-), U5.4 (V-), U5.6 (-)
