File: aix_amp/interface.kicad_sch (KiCad schematic)
At the start: 6 parts, among them J2 4pin_output, J3 3pin_output, J4 aux_input, J5 USB_C_Receptacle

Commit message: 앰프 기본 완성
Parts:
- removed D4: 1N4148WT, Diode_SMD:D_SOD-523, symbol Diode:1N4148WT
Connections:
- net +5V renamed +5V_in
Changed lines of the file:
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@@
 		(color 0 0 0 0)
 	)
-	(junction
-		(at 231.14 68.58)
-		(diameter 0)
-		(color 0 0 0 0)
-	)
 	(no_connect
 		(at 242.57 53.34)
@@
 	(wire
 		(pts
-			(xy 219.71 68.58) (xy 213.36 68.58)
-		)
-		(stroke
-			(width 0)
-			(type default)
-		)
-	)
-	(wire
-		(pts
 			(xy 43.18 138.43) (xy 66.04 138.43)
 		)
@@
 	(wire
 		(pts
-			(xy 213.36 68.58) (xy 213.36 69.85)
-		)
-		(stroke
-			(width 0)
-			(type default)
-		)
-	)
-	(wire
-		(pts
 			(xy 248.92 93.98) (xy 240.03 93.98)
 		)
@@
 		(pts
 			(xy 58.42 29.21) (xy 58.42 46.99)
-		)
-		(stroke
-			(width 0)
-			(type default)
-		)
-	)
-	(wire
-		(pts
-			(xy 231.14 68.58) (xy 227.33 68.58)
 		)
 		(stroke
@@
 			(justify left bottom)
 		)
-		(property "Netclass" "mic_input"
+		(property "Netclass" "mic_out"
 			(at 84.5185 121.92 0)
 			(effects
@@
 				(path "/92363970-7a70-4a9d-91f1-fb8480a3037e/0efb2e7e-752a-4c09-a01b-8352ef63af5b"
 					(reference "J4")
-					(unit 1)
-				)
-			)
-		)
-	)
-	(symbol
-		(lib_id "power:GND")
-		(at 213.36 69.85 0)
-		(unit 1)
-		(exclude_from_sim no)
-		(in_bom yes)
-		(on_board yes)
-		(dnp no)
-		(fields_autoplaced yes)
-		(property "Reference" "#PWR09"
-			(at 213.36 76.2 0)
-			(effects
-				(font
-					(size 1.27 1.27)
-				)
-				(hide yes)
-			)
-		)
-		(property "Value" "GND"
-			(at 213.36 74.93 0)
-			(effects
-				(font
-					(size 1.27 1.27)
-				)
-			)
-		)
-		(property "Footprint" ""
-			(at 213.36 69.85 0)
-			(effects
-				(font
-					(size 1.27 1.27)
-				)
-				(hide yes)
-			)
-		)
-		(property "Datasheet" ""
-			(at 213.36 69.85 0)
-			(effects
-				(font
-					(size 1.27 1.27)
-				)
-				(hide yes)
-			)
-		)
-		(property "Description" "Power symbol creates a global label with name \"GND\" , ground"
-			(at 213.36 69.85 0)
-			(effects
-				(font
-					(size 1.27 1.27)
-				)
-				(hide yes)
-			)
-		)
-		(pin "1"
-		)
-		(instances
-			(project ""
-				(path "/92363970-7a70-4a9d-91f1-fb8480a3037e/0efb2e7e-752a-4c09-a01b-8352ef63af5b"
-					(reference "#PWR09")
 					(unit 1)
 				)
@@
 	)
 	(symbol
-		(lib_id "Diode:1N4148WT")
-		(at 223.52 68.58 0)
-		(unit 1)
-		(exclude_from_sim no)
-		(in_bom yes)
-		(on_board yes)
-		(dnp no)
-		(property "Reference" "D4"
-			(at 223.52 74.93 0)
-			(effects
-				(font
-					(size 1.27 1.27)
-				)
-			)
-		)
-		(property "Value" "1N4148WT"
-			(at 223.52 72.39 0)
-			(effects
-				(font
-					(size 1.27 1.27)
-				)
-			)
-		)
-		(property "Footprint" "Diode_SMD:D_SOD-523"
-			(at 223.52 73.025 0)
-			(effects
-				(font
-					(size 1.27 1.27)
-				)
-				(hide yes)
-			)
-		)
-		(property "Datasheet" "https://www.diodes.com/assets/Datasheets/ds30396.pdf"
-			(at 223.52 68.58 0)
-			(effects
-				(font
-					(size 1.27 1.27)
-				)
-				(hide yes)
-			)
-		)
-		(property "Description" "75V 0.15A Fast switching Diode, SOD-523"
-			(at 223.52 68.58 0)
-			(effects
-				(font
-					(size 1.27 1.27)
-				)
-				(hide yes)
-			)
-		)
-		(property "Sim.Device" "D"
-			(at 223.52 68.58 0)
-			(effects
-				(font
-					(size 1.27 1.27)
-				)
-				(hide yes)
-			)
-		)
-		(property "Sim.Pins" "1=K 2=A"
-			(at 223.52 68.58 0)
-			(effects
-				(font
-					(size 1.27 1.27)
-				)
-				(hide yes)
-			)
-		)
-		(pin "1"
-		)
-		(pin "2"
-		)
-		(instances
-			(project ""
-				(path "/92363970-7a70-4a9d-91f1-fb8480a3037e/0efb2e7e-752a-4c09-a01b-8352ef63af5b"
-					(reference "D4")
-					(unit 1)
-				)
-			)
-		)
-	)
-	(symbol
 		(lib_id "power:GND")
 		(at 231.14 68.58 0)
@@
 			)
 		)
-		(property "Value" "+5V"
-			(at 76.2 59.69 0)
-			(effects
-				(font
-					(size 1.27 1.27)
-				)
-			)
-		)
+		(property "Value" "+5V_in"
+			(at 78.74 63.4999 0)
+			(effects
+				(font
+					(size 1.27 1.27)
+				)
+				(justify left)
+			)
+		)
